File: Hardware/rele wifi pwoss - copia.kicad_pcb (KiCad board)
At the start: 2 copper layers, 47 parts, among them IC1 MC7805CD2TG, J1 BORNERA, J2 BORNERA, J3 Conn_01x04_Pin, J4 BORNERA, J5 BORNERA, K3 SANYOU_SRD_Form_C, K6 SANYOU_SRD_Form_C, K7 SANYOU_SRD_Form_C, K8 SANYOU_SRD_Form_C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

Commit message: Add files via upload
Parts:
- removed J3: Conn_01x04_Pin, Connector_PinSocket_2.54mm:PinSocket_1x04_P2.54mm_Vertical
- Q1, Q2, Q4, Q5: footprint Package_TO_SOT_SMD:SOT-23 -> bc547:SOT95P230X110-3N
- moved BORNERA1 25.8 mm to (71.7, 127.7), turned to 0 degrees
- moved C2 8.68 mm to (51.1, 110.0)
- moved U7 5.25 mm to (63.8, 74.4)
- moved C1 4.46 mm to (64.8, 117.5)
- moved H3 4.01 mm to (50.7, 127.0)
- moved H4 4.00 mm to (142.2, 127.0)
- moved SW1 3.22 mm to (76.8, 120.0)
- moved IC1 3.04 mm to (63.2, 103.0)
- moved R13 0.57 mm to (85.5, 114.3)
- moved R10 0.48 mm to (85.5, 95.0)
- moved J5 0.47 mm to (133.7, 105.7)
- moved R2 0.40 mm to (85.5, 75.8)
- moved R3 0.33 mm to (85.5, 56.9)
- moved R11 0.07 mm to (85.5, 85.5)
- moved U4 0.07 mm to (92.0, 89.0)
Connections:
- D1 pad 2: RELE-2 -> ESP32 IO22
- D3 pad 2: RELE-4 -> ESP32 IO23
- D7 pad 2: RELE-1 ->  ESP32 IO21
- D9 pad 2: RELE-3 -> ESP32 IO19
- R1 pad 1: RELE-4 -> ESP32 IO23
- R11 pad 1: RELE-1 ->  ESP32 IO21
- R14 pad 1: RELE-3 -> ESP32 IO19
- R5 pad 1: RELE-2 -> ESP32 IO22
- U7 pad 27: RELE-3 -> unconnected-(U7-IO16-Pad27)
- U7 pad 28: RELE-1 -> unconnected-(U7-IO17-Pad28)
- U7 pad 30: RELE-2 -> unconnected-(U7-IO18-Pad30)
- U7 pad 31: RELE-4 -> ESP32 IO19
- U7 pad 33: PIN-2 ->  ESP32 IO21
- U7 pad 36: PIN-1 -> ESP32 IO22
- U7 pad 37: unconnected-(U7-IO23-Pad37) -> ESP32 IO23
Routing:
- net +5V: track 78.1 -> 21.4 mm
- net ESP32 IO19: track 0.00 -> 44.8 mm
- net RELE-4: track 32.0 -> 0.00 mm
- net PIN-2: track 31.5 -> 0.00 mm
- net  ESP32 IO21: track 0.00 -> 31.5 mm
- net RELE-3: track 30.6 -> 0.00 mm
- net PIN-1: track 22.9 -> 0.00 mm
- net ESP32 IO22: track 0.00 -> 19.1 mm
- net Net-(BORNERA1-Pin_2): track 25.2 -> 7.72 mm
- net ESP32 IO23: track 0.00 -> 16.6 mm
- net RELE-2: track 15.8 -> 0.00 mm
- net RELE-1: track 14.2 -> 0.00 mm
- net VCC: track 388.7 -> 398.7 mm
- net Net-(U1-A): track 5.23 -> 4.34 mm
- net Net-(D9-K): track 2.25 -> 2.81 mm
