File: Hardware/rele wifi pwoss.kicad_pcb (KiCad board)
At the start: 2 copper layers, 47 parts, among them IC1 MC7805CD2TG, J1 BORNERA, J2 BORNERA, J3 Conn_01x04_Pin, J4 BORNERA, J5 BORNERA, K3 SANYOU_SRD_Form_C, K6 SANYOU_SRD_Form_C, K7 SANYOU_SRD_Form_C, K8 SANYOU_SRD_Form_C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

Commit message: Add files via upload
ULTIMO AVANCE DE PCB Y ESQUEMATICO 12/8/25
Parts:
- removed Q2, Q4: BC547, Package_TO_SOT_SMD:SOT-23
- added Q3: MMBT2222A, Package_TO_SOT_SMD:SOT-23, B.Cu at (72.7, 91.9)
- added Q6: MMBT2222A, Package_TO_SOT_SMD:SOT-23, B.Cu at (72.7, 34.8)
- Q1, Q5: value BC547 -> MMBT2222A
- moved Q5 48.6 mm to (72.0, 72.7), turned to 0 degrees
- moved C1 35.8 mm to (38.8, 93.3)
- moved C2 35.8 mm to (30.7, 89.1)
- moved D2 35.8 mm to (76.5, 32.8)
- moved H3 35.8 mm to (21.5, 102.1)
- moved IC1 35.8 mm to (37.2, 82.1)
- moved J1 35.8 mm to (104.9, 27.6)
- moved J2 35.8 mm to (104.9, 46.4)
- moved J3 35.8 mm to (30.7, 25.6)
- moved J4 35.8 mm to (104.8, 65.6)
- moved J5 35.8 mm to (104.7, 85.3)
- moved K3 35.8 mm to (80.6, 32.8)
- moved SW1 35.8 mm to (47.7, 95.9)
- moved U7 35.8 mm to (34.8, 58.8)
- moved D10 35.8 mm to (77.7, 89.9)
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Connections:
- Q1 pad 1: Net-(D4-A) -> Net-(Q1-B)
- Q1 pad 2: Net-(Q1-B) -> GND
- Q1 pad 3: GND -> Net-(D4-A)
- Q5 pad 1: Net-(D10-A) -> Net-(Q5-B)
- Q5 pad 2: Net-(Q5-B) -> GND
- Q5 pad 3: GND -> Net-(D8-A)
- R12 pad 2: Net-(Q4-B) -> Net-(Q5-B)
- R15 pad 2: Net-(Q5-B) -> Net-(Q3-B)
Routing:
- net VCC: track 388.7 -> 227.3 mm
- net GND: track 0.00 -> 63.5 mm, vias 0 -> 5
- net Net-(Q3-B): track 0.00 -> 3.15 mm
- net Net-(Q4-B): track 2.27 -> 0.00 mm
- net Net-(Q1-B): track 2.14 -> 3.15 mm
- net Net-(D10-A): track 14.0 -> 13.0 mm
- net Net-(Q6-B): track 2.16 -> 3.15 mm
- net Net-(D4-A): track 13.5 -> 12.5 mm
- net Net-(D2-A): track 13.3 -> 12.3 mm
- net RELE-3: track 30.6 -> 31.3 mm
- net RELE-4: track 32.0 -> 31.5 mm
- net RELE-2: track 15.8 -> 15.3 mm
Other:
- board outline added: 99.9 x 86.8 mm
