File: Hardware/uwo.kicad_pcb (KiCad board)
At the start: 2 copper layers, 99.9 x 86.8 mm, 47 parts, among them IC1 MC7805CD2TG, J1 BORNERA, J2 BORNERA, J3 Conn_01x04_Pin, J4 BORNERA, J5 BORNERA, K3 SANYOU_SRD_Form_C, K6 SANYOU_SRD_Form_C, K7 SANYOU_SRD_Form_C, K8 SANYOU_SRD_Form_C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

Commit message: Add files via upload
ULTIMO AVANCE DEL RELE WIFI 12/8/2025 "UWO"
Routing:
- net (no net): track 0.00 -> 63.8 mm, vias 0 -> 5
Changed lines of the file:
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@@
 		(property ki_fp_filters "TerminalBlock*:*")
 		(sheetname "/")
-		(sheetfile "rele wifi pwoss.kicad_sch")
+		(sheetfile "uwo.kicad_sch")
 		(attr through_hole)
 		(fp_line
@@
 		(property ki_fp_filters "TerminalBlock*:*")
 		(sheetname "/")
-		(sheetfile "rele wifi pwoss.kicad_sch")
+		(sheetfile "uwo.kicad_sch")
 		(attr through_hole)
 		(fp_line
@@
 		(property ki_fp_filters "TerminalBlock*:*")
 		(sheetname "/")
-		(sheetfile "rele wifi pwoss.kicad_sch")
+		(sheetfile "uwo.kicad_sch")
 		(attr through_hole)
 		(fp_line
@@
 		(property ki_fp_filters "Relay*SPDT*SANYOU*SRD*Series*Form*C*")
 		(sheetname "/")
-		(sheetfile "rele wifi pwoss.kicad_sch")
+		(sheetfile "uwo.kicad_sch")
 		(attr through_hole)
 		(fp_line
@@
 		(property ki_fp_filters "MountingHole*")
 		(sheetname "/")
-		(sheetfile "rele wifi pwoss.kicad_sch")
+		(sheetfile "uwo.kicad_sch")
 		(attr exclude_from_pos_files exclude_from_bom)
 		(fp_circle
@@
 		(property ki_fp_filters "Relay*SPDT*SANYOU*SRD*Series*Form*C*")
 		(sheetname "/")
-		(sheetfile "rele wifi pwoss.kicad_sch")
+		(sheetfile "uwo.kicad_sch")
 		(attr through_hole)
 		(fp_line
@@
 		(property ki_fp_filters "Relay*SPDT*SANYOU*SRD*Series*Form*C*")
 		(sheetname "/")
-		(sheetfile "rele wifi pwoss.kicad_sch")
+		(sheetfile "uwo.kicad_sch")
 		(attr through_hole)
 		(fp_line
@@
 		(property ki_fp_filters "Connector*:*_1x??_*")
 		(sheetname "/")
-		(sheetfile "rele wifi pwoss.kicad_sch")
+		(sheetfile "uwo.kicad_sch")
 		(attr through_hole)
 		(fp_line
@@
 		)
 		(sheetname "/")
-		(sheetfile "rele wifi pwoss.kicad_sch")
+		(sheetfile "uwo.kicad_sch")
 		(attr through_hole)
 		(fp_line
@@
 		(property ki_fp_filters "MountingHole*")
 		(sheetname "/")
-		(sheetfile "rele wifi pwoss.kicad_sch")
+		(sheetfile "uwo.kicad_sch")
 		(attr exclude_from_pos_files exclude_from_bom)
 		(fp_circle
@@
 		(property ki_fp_filters "TerminalBlock*:*")
 		(sheetname "/")
-		(sheetfile "rele wifi pwoss.kicad_sch")
+		(sheetfile "uwo.kicad_sch")
 		(attr through_hole)
 		(fp_line
@@
 		(property ki_fp_filters "MountingHole*")
 		(sheetname "/")
-		(sheetfile "rele wifi pwoss.kicad_sch")
+		(sheetfile "uwo.kicad_sch")
 		(attr exclude_from_pos_files exclude_from_bom)
 		(fp_circle
@@
 		)
 		(sheetname "/")
-		(sheetfile "rele wifi pwoss.kicad_sch")
+		(sheetfile "uwo.kicad_sch")
 		(attr through_hole)
 		(fp_line
@@
 		(property ki_fp_filters "Connector*:*_1x??_*")
 		(sheetname "/")
-		(sheetfile "rele wifi pwoss.kicad_sch")
+		(sheetfile "uwo.kicad_sch")
 		(attr through_hole)
 		(fp_line
@@
 		(property ki_fp_filters "MountingHole*")
 		(sheetname "/")
-		(sheetfile "rele wifi pwoss.kicad_sch")
+		(sheetfile "uwo.kicad_sch")
 		(attr exclude_from_pos_files exclude_from_bom)
 		(fp_circle
@@
 		(property ki_fp_filters "Relay*SPDT*SANYOU*SRD*Series*Form*C*")
 		(sheetname "/")
-		(sheetfile "rele wifi pwoss.kicad_sch")
+		(sheetfile "uwo.kicad_sch")
 		(attr through_hole)
 		(fp_line
@@
 		(property ki_fp_filters "R_*")
 		(sheetname "/")
-		(sheetfile "rele wifi pwoss.kicad_sch")
+		(sheetfile "uwo.kicad_sch")
 		(attr smd)
 		(fp_line
@@
 		(property ki_fp_filters "R_*")
 		(sheetname "/")
-		(sheetfile "rele wifi pwoss.kicad_sch")
+		(sheetfile "uwo.kicad_sch")
 		(attr smd)
 		(fp_line
@@
 		(property ki_fp_filters "SOT?23*")
 		(sheetname "/")
-		(sheetfile "rele wifi pwoss.kicad_sch")
+		(sheetfile "uwo.kicad_sch")
 		(attr smd)
 		(fp_line
@@
 		(property ki_fp_filters "SOT?23*")
 		(sheetname "/")
-		(sheetfile "rele wifi pwoss.kicad_sch")
+		(sheetfile "uwo.kicad_sch")
 		(attr smd)
 		(fp_line
@@
 		)
 		(sheetname "/")
-		(sheetfile "rele wifi pwoss.kicad_sch")
+		(sheetfile "uwo.kicad_sch")
 		(attr smd)
 		(fp_line
@@
 		)
 		(sheetname "/")
-		(sheetfile "rele wifi pwoss.kicad_sch")
+		(sheetfile "uwo.kicad_sch")
 		(attr smd)
 		(fp_line
@@
 		(property ki_fp_filters "TO-???* *_Diode_* *SingleDiode* D_*")
 		(sheetname "/")
-		(sheetfile "rele wifi pwoss.kicad_sch")
+		(sheetfile "uwo.kicad_sch")
 		(attr smd)
 		(fp_line
@@
 		(property ki_fp_filters "LED* LED_SMD:* LED_THT:*")
 		(sheetname "/")
-		(sheetfile "rele wifi pwoss.kicad_sch")
+		(sheetfile "uwo.kicad_sch")
 		(attr smd)
 		(fp_line
@@
 		(property ki_fp_filters "LED* LED_SMD:* LED_THT:*")
 		(sheetname "/")
-		(sheetfile "rele wifi pwoss.kicad_sch")
+		(sheetfile "uwo.kicad_sch")
 		(attr smd)
 		(fp_line
@@
 		(property ki_fp_filters "R_*")
 		(sheetname "/")
-		(sheetfile "rele wifi pwoss.kicad_sch")
+		(sheetfile "uwo.kicad_sch")
 		(attr smd)
 		(fp_line
@@
 		(property ki_fp_filters "SOT?23*")
 		(sheetname "/")
-		(sheetfile "rele wifi pwoss.kicad_sch")
+		(sheetfile "uwo.kicad_sch")
 		(attr smd)
 		(fp_line
@@
 		(property ki_fp_filters "TO-???* *_Diode_* *SingleDiode* D_*")
 		(sheetname "/")
-		(sheetfile "rele wifi pwoss.kicad_sch")
+		(sheetfile "uwo.kicad_sch")
 		(attr smd)
 		(fp_line
@@
 		(property ki_fp_filters "R_*")
 		(sheetname "/")
-		(sheetfile "rele wifi pwoss.kicad_sch")
+		(sheetfile "uwo.kicad_sch")
 		(attr smd)
 		(fp_line
@@
 		(property ki_fp_filters "R_*")
 		(sheetname "/")
-		(sheetfile "rele wifi pwoss.kicad_sch")
+		(sheetfile "uwo.kicad_sch")
 		(attr smd)
 		(fp_line
@@
 		(property ki_fp_filters "SOT?23*")
 		(sheetname "/")
-		(sheetfile "rele wifi pwoss.kicad_sch")
+		(sheetfile "uwo.kicad_sch")
 		(attr smd)
 		(fp_line
@@
 		)
 		(sheetname "/")
-		(sheetfile "rele wifi pwoss.kicad_sch")
+		(sheetfile "uwo.kicad_sch")
 		(attr smd)
 		(fp_line
@@
 		(property ki_fp_filters "C_*")
 		(sheetname "/")
-		(sheetfile "rele wifi pwoss.kicad_sch")
+		(sheetfile "uwo.kicad_sch")
 		(attr smd)
 		(fp_line
@@
 		(property ki_fp_filters "R_*")
 		(sheetname "/")
-		(sheetfile "rele wifi pwoss.kicad_sch")
+		(sheetfile "uwo.kicad_sch")
 		(attr smd)
 		(fp_line
@@
 		(property ki_fp_filters "LED* LED_SMD:* LED_THT:*")
 		(sheetname "/")
-		(sheetfile "rele wifi pwoss.kicad_sch")
+		(sheetfile "uwo.kicad_sch")
 		(attr smd)
 		(fp_line
@@
 		(property ki_fp_filters "R_*")
 		(sheetname "/")
-		(sheetfile "rele wifi pwoss.kicad_sch")
+		(sheetfile "uwo.kicad_sch")
 		(attr smd)
 		(fp_line
@@
 		(property ki_fp_filters "TO-???* *_Diode_* *SingleDiode* D_*")
 		(sheetname "/")
-		(sheetfile "rele wifi pwoss.kicad_sch")
+		(sheetfile "uwo.kicad_sch")
 		(attr smd)
 		(fp_line
@@
 		)
 		(sheetname "/")
-		(sheetfile "rele wifi pwoss.kicad_sch")
+		(sheetfile "uwo.kicad_sch")
 		(attr smd)
 		(fp_line
@@
 		(property ki_fp_filters "TO-???* *_Diode_* *SingleDiode* D_*")
 		(sheetname "/")
-		(sheetfile "rele wifi pwoss.kicad_sch")
+		(sheetfile "uwo.kicad_sch")
 		(attr smd)
 		(fp_line
@@
 		(property ki_fp_filters "R_*")
 		(sheetname "/")
-		(sheetfile "rele wifi pwoss.kicad_sch")
+		(sheetfile "uwo.kicad_sch")
 		(attr smd)
 		(fp_line
@@
 		(property ki_fp_filters "LED* LED_SMD:* LED_THT:*")
 		(sheetname "/")
-		(sheetfile "rele wifi pwoss.kicad_sch")
+		(sheetfile "uwo.kicad_sch")
 		(attr smd)
 		(fp_line
@@
 		(property ki_fp_filters "C_*")
 		(sheetname "/")
-		(sheetfile "rele wifi pwoss.kicad_sch")
+		(sheetfile "uwo.kicad_sch")
 		(attr smd)
 		(fp_line
@@
 		(property ki_fp_filters "R_*")
 		(sheetname "/")
-		(sheetfile "rele wifi pwoss.kicad_sch")
+		(sheetfile "uwo.kicad_sch")
 		(attr smd)
 		(fp_line
@@
 		(property ki_fp_filters "R_*")
 		(sheetname "/")
-		(sheetfile "rele wifi pwoss.kicad_sch")
+		(sheetfile "uwo.kicad_sch")
 		(attr smd)
 		(fp_line
@@
 		(property ki_fp_filters "R_*")
 		(sheetname "/")
-		(sheetfile "rele wifi pwoss.kicad_sch")
+		(sheetfile "uwo.kicad_sch")
 		(attr smd)
 		(fp_line
@@
 		(property ki_fp_filters "R_*")
 		(sheetname "/")
-		(sheetfile "rele wifi pwoss.kicad_sch")
+		(sheetfile "uwo.kicad_sch")
 		(attr smd)
 		(fp_line
@@
 		)
 		(sheetname "/")
-		(sheetfile "rele wifi pwoss.kicad_sch")
+		(sheetfile "uwo.kicad_sch")
 		(attr smd)
 		(fp_line
@@
 	)
 	(segment
+		(start 97.75 92)
+		(end 97.75 72.75)
+		(width 1)
+		(layer "F.Cu")
+		(net 0)
+	)
+	(segment
+		(start 97.75 72.75)
+		(end 97.75 54)
+		(width 1)
+		(layer "F.Cu")
+		(net 0)
+	)
+	(segment
+		(start 97.75 54)
+		(end 97.75 47.5)
+		(width 1)
+		(layer "F.Cu")
+		(net 0)
+	)
+	(segment
+		(start 97.75 111.25)
+		(end 97.75 92)
+		(width 1)
+		(layer "F.Cu")
+		(net 0)
+	)
+	(via
+		(at 97.75 54)
+		(size 1)
+		(drill 0.4)
+		(layers "F.Cu" "B.Cu")
+		(net 0)
+	)
+	(via
+		(at 97.75 47.5)
+		(size 1)
+		(drill 0.4)
+		(layers "F.Cu" "B.Cu")
+		(net 0)
+	)
+	(via
+		(at 97.75 92)
+		(size 1)
+		(drill 0.4)
+		(layers "F.Cu" "B.Cu")
+		(net 0)
+	)
+	(via
+		(at 97.75 111.25)
+		(size 1)
+		(drill 0.4)
+		(layers "F.Cu" "B.Cu")
+		(net 0)
+	)
+	(via
+		(at 97.75 72.75)
+		(size 1)
+		(drill 0.4)
+		(layers "F.Cu" "B.Cu")
+		(net 0)
+	)
+	(segment
