File: Diseño-3D/uwo.kicad_pcb (KiCad board)
At the start: 2 copper layers, 47 parts, among them IC1 MC7805CD2TG, J1 BORNERA, J2 BORNERA, J3 Conn_01x04_Pin, J4 BORNERA, J5 BORNERA, K3 SANYOU_SRD_Form_C, K6 SANYOU_SRD_Form_C, K7 SANYOU_SRD_Form_C, K8 SANYOU_SRD_Form_C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

Commit message: Add files via upload
Parts:
- U7: footprint EESTN5:ESP32_DEVKITC -> ESP32:MODULE_ESP32-DEVKITC
- moved IC1 1.22 mm to (66.2, 103.0)
- moved C1 0.90 mm to (67.8, 114.2)
- moved C2 0.70 mm to (59.8, 110.0)
- moved U7 0.24 mm to (63.8, 79.7), turned to 0 degrees
Routing:
- net VCC: track 389.1 -> 387.7 mm
- net +5V: track 76.6 -> 78.1 mm
