File: Diseño-3D/uwo.kicad_sch (KiCad schematic)
At the start: 47 parts, among them IC1 MC7805CD2TG, J1 BORNERA, J2 BORNERA, J3 Conn_01x04_Pin, J4 BORNERA, J5 BORNERA, K3 SANYOU_SRD_Form_C, K6 SANYOU_SRD_Form_C, K7 SANYOU_SRD_Form_C, K8 SANYOU_SRD_Form_C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

Commit message: Add files via upload
Parts:
- U7: footprint EESTN5:ESP32_DEVKITC -> ESP32:MODULE_ESP32-DEVKITC
Changed lines of the file:
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@@
 			)
 		)
-		(property "Footprint" "EESTN5:ESP32_DEVKITC"
+		(property "Footprint" "ESP32:MODULE_ESP32-DEVKITC"
 			(at 44.45 48.26 0)
 			(effects
